Commit message: 参考GitHub项目lmark1/velodyne_simulator，为本项目添加了3D激光雷达模拟的xacro描述文件，以及一个publish PointCloud2数据类型的topic的gezebo插件程序

File: urdf/MarsRover.xacro (robot description, xacro)
@@ -849,5 +849,5 @@
       velocity="0" />
   </joint>
-  <link
+  <!--link
     name="LiDAR">
     <inertial>
@@ -899,7 +899,11 @@
     <child
       link="LiDAR" />
-    <!--axis
-      xyz="0 1 0" /-->
-  </joint>
+    <axis
+      xyz="0 1 0" />
+  </joint-->
+  <xacro:include filename="$(find MarsRover)/urdf/PandarQT.xacro"/>
+  <PandarQT parent="LiDARSupport" name="PandarQT" topic="PandarQT_Data" hz="10" lasers="64" samples="600" visual="false">
+    <origin xyz="-0.0375 0.0544 0" rpy="${-PI/2} 0 0" />
+  </PandarQT>
   <!--TRANSMISSION-->
   <!--transmission name="simple_trans">

Commit message: 删除了被注释掉的无用的代码，使用rviz订阅激光雷达数据topic并显示，添加了libgazebo_ros_joint_state_publisher.so插件使rviz可同步显示gazebo中火星车的各个关节状态

File: urdf/MarsRover.xacro (robot description, xacro)
@@ -5,16 +5,13 @@
 <robot xmlns:xacro="http://www.ros.org/wiki/xacro"
   name="MarsRover">
-  <xacro:include filename="$(find MarsRover)/urdf/MarsRover.gazebo" />
+  <xacro:include filename="$(find mars_rover)/urdf/MarsRover.gazebo" />
   <xacro:property name="PI" value="3.141592654" />
-  <xacro:property name="LidarAngle" value="${0}" />
+  <xacro:property name="LidarAngle" value="${PI/6}" />
   <xacro:property name="LidarHeight" value="-0.0" />
-  <link
-    name="body">
-    <inertial>
-      <origin
-        xyz="-0.000147897244928197 -0.0822271126898096 1.11022302462516E-16"
-        rpy="0 0 0" />
-      <mass
-        value="32.9286570826472" />
+  <xacro:property name="LidarName" value="PandarQT" />
+  <link name="body">
+    <inertial>
+      <origin xyz="-0.000147897244928197 -0.0822271126898096 1.11022302462516E-16" rpy="0 0 0" />
+      <mass value="32.9286570826472" />
       <inertia
         ixx="4.47491142188154"
@@ -26,24 +23,16 @@
     </inertial>
     <visual>
-      <origin
-        xyz="0 0 0"
-        rpy="0 0 0" />
-      <geometry>
-        <mesh
-          filename="package://MarsRover/meshes/body.STL" />
-      </geometry>
-      <material
-        name="">
-        <color
-          rgba="0.752941176470588 0.752941176470588 0.752941176470588 1" />
-      </material>
-    </visual>
-    <collision>
-      <origin
-        xyz="0 0 0"
-        rpy="0 0 0" />
-      <geometry>
-        <mesh
-          filename="package://MarsRover/meshes/body.STL" />
+      <origin xyz="0 0 0" rpy="0 0 0" />
+      <geometry>
+        <mesh filename="package://mars_rover/meshes/body.STL" />
+      </geometry>
+      <material name="">
+        <color rgba="0.752941176470588 0.752941176470588 0.752941176470588 1" />
+      </material>
+    </visual>
+    <collision>
+      <origin xyz="0 0 0" rpy="0 0 0" />
+      <geometry>
+        <mesh filename="package://mars_rover/meshes/body.STL" />
       </geometry>
     </collision>
@@ -52,9 +41,6 @@
     name="DiffBar">
     <inertial>
-      <origin
-        xyz="7.23369697475107E-10 -0.0223125966605722 3.3729640969149E-08"
-        rpy="0 0 0" />
-      <mass
-        value="1.49170112220708" />
+      <origin xyz="7.23369697475107E-10 -0.0223125966605722 3.3729640969149E-08" rpy="0 0 0" />
+      <mass value="1.49170112220708" />
       <inertia
         ixx="0.030385701616174"
@@ -66,48 +52,29 @@
     </inertial>
     <visual>
-      <origin
-        xyz="0 0 0"
-        rpy="0 0 0" />
-      <geometry>
-        <mesh
-          filename="package://MarsRover/meshes/DiffBar.STL" />
-      </geometry>
-      <material
-        name="">
-        <color
-          rgba="0.898039215686275 0.917647058823529 0.929411764705882 1" />
-      </material>
-    </visual>
-    <collision>
-      <origin
-        xyz="0 0 0"
-        rpy="0 0 0" />
-      <geometry>
-        <mesh
-          filename="package://MarsRover/meshes/DiffBar.STL" />
-      </geometry>
-    </collision>
-  </link>
-  <joint
-    name="joint_body_DiffBar"
-    type="continuous">
-    <origin
-      xyz="0.20043 -0.225 0"
-      rpy="0 0 0" />
-    <parent
-      link="body" />
-    <child
-      link="DiffBar" />
-    <axis
-      xyz="0 1 0" />
-  </joint>
-  <link
-    name="LeftMainRocker">
-    <inertial>
-      <origin
-        xyz="0.194777234245267 -0.101638011239522 -0.0322190943393932"
-        rpy="0 0 0" />
-      <mass
-        value="2.31659033764537" />
+      <origin xyz="0 0 0" rpy="0 0 0" />
+      <geometry>
+        <mesh filename="package://mars_rover/meshes/DiffBar.STL" />
+      </geometry>
+      <material name="">
+        <color rgba="0.898039215686275 0.917647058823529 0.929411764705882 1" />
+      </material>
+    </visual>
+    <collision>
+      <origin xyz="0 0 0" rpy="0 0 0" />
+      <geometry>
+        <mesh filename="package://mars_rover/meshes/DiffBar.STL" />
+      </geometry>
+    </collision>
+  </link>
+  <joint name="joint_body_DiffBar" type="continuous">
+    <origin xyz="0.20043 -0.225 0" rpy="0 0 0" />
+    <parent link="body" />
+    <child link="DiffBar" />
+    <axis xyz="0 1 0" />
+  </joint>
+  <link name="LeftMainRocker">
+    <inertial>
+      <origin xyz="0.194777234245267 -0.101638011239522 -0.0322190943393932" rpy="0 0 0" />
+      <mass value="2.31659033764537" />
       <inertia
         ixx="0.0253182901443958"
@@ -119,48 +86,31 @@
     </inertial>
     <visual>
-      <origin
-        xyz="0 0 0"
-        rpy="0 0 0" />
-      <geometry>
-        <mesh
-          filename="package://MarsRover/meshes/LeftMainRocker.STL" />
-      </geometry>
-      <material
-        name="">
-        <color
-          rgba="0.792156862745098 0.819607843137255 0.933333333333333 1" />
-      </material>
-    </visual>
-    <collision>
-      <origin
-        xyz="0 0 0"
-        rpy="0 0 0" />
-      <geometry>
-        <mesh
-          filename="package://MarsRover/meshes/LeftMainRocker.STL" />
-      </geometry>
-    </collision>
-  </link>
-  <joint
-    name="joint_body_LeftMainRocker"
-    type="continuous">
-    <origin
-      xyz="0 -0.155 -0.395"
-      rpy="0 0 0" />
-    <parent
-      link="body" />
-    <child
-      link="LeftMainRocker" />
-    <axis
-      xyz="0 0 1" />
-  </joint>
-  <link
-    name="LeftViceRocker">
+      <origin xyz="0 0 0" rpy="0 0 0" />
+      <geometry>
+        <mesh filename="package://mars_rover/meshes/LeftMainRocker.STL" />
+      </geometry>
+      <material name="">
+        <color rgba="0.792156862745098 0.819607843137255 0.933333333333333 1" />
+      </material>
+    </visual>
+    <collision>
+      <origin xyz="0 0 0" rpy="0 0 0" />
+      <geometry>
+        <mesh filename="package://mars_rover/meshes/LeftMainRocker.STL" />
+      </geometry>
+    </collision>
+  </link>
+  <joint name="joint_body_LeftMainRocker" type="continuous">
+    <origin xyz="0 -0.155 -0.395" rpy="0 0 0" />
+    <parent link="body" />
+    <child link="LeftMainRocker" />
+    <axis xyz="0 0 1" />
+  </joint>
+  <link name="LeftViceRocker">
     <inertial>
       <origin
         xyz="0.000324935586217618 -0.142828935520301 -0.00457781208829167"
         rpy="0 0 0" />
-      <mass
-        value="1.70193743881046" />
+      <mass value="1.70193743881046" />
       <inertia
         ixx="0.011640762472159"
@@ -172,48 +122,29 @@
     </inertial>
     <visual>
-      <origin
-        xyz="0 0 0"
-        rpy="0 0 0" />
-      <geometry>
-        <mesh
-          filename="package://MarsRover/meshes/LeftViceRocker.STL" />
-      </geometry>
-      <material
-        name="">
-        <color
-          rgba="0.792156862745098 0.819607843137255 0.933333333333333 1" />
-      </material>
-    </visual>
-    <collision>
-      <origin
-        xyz="0 0 0"
-        rpy="0 0 0" />
-      <geometry>
-        <mesh
-          filename="package://MarsRover/meshes/LeftViceRocker.STL" />
-      </geometry>
-    </collision>
-  </link>
-  <joint
-    name="joint_LeftMainRocker_LeftViceRocker"
-    type="continuous">
-    <origin
-      xyz="-0.40088 -0.023072 -0.055"
-      rpy="0 0 0" />
-    <parent
-      link="LeftMainRocker" />
-    <child
-      link="LeftViceRocker" />
-    <axis
-      xyz="0 0 1" />
-  </joint>
-  <link
-    name="LeftMiddleWheel">
-    <inertial>
-      <origin
-        xyz="0 -2.77555756156289E-17 1.66533453693773E-16"
-        rpy="0 0 0" />
-      <mass
-        value="2.46800319485063" />
+      <origin xyz="0 0 0" rpy="0 0 0" />
+      <geometry>
+        <mesh filename="package://mars_rover/meshes/LeftViceRocker.STL" />
+      </geometry>
+      <material name="">
+        <color rgba="0.792156862745098 0.819607843137255 0.933333333333333 1" />
+      </material>
+    </visual>
+    <collision>
+      <origin xyz="0 0 0" rpy="0 0 0" />
+      <geometry>
+        <mesh filename="package://mars_rover/meshes/LeftViceRocker.STL" />
+      </geometry>
+    </collision>
+  </link>
+  <joint name="joint_LeftMainRocker_LeftViceRocker" type="continuous">
+    <origin xyz="-0.40088 -0.023072 -0.055" rpy="0 0 0" />
+    <parent link="LeftMainRocker" />
+    <child link="LeftViceRocker" />
+    <axis xyz="0 0 1" />
+  </joint>
+  <link name="LeftMiddleWheel">
+    <inertial>
+      <origin xyz="0 -2.77555756156289E-17 1.66533453693773E-16" rpy="0 0 0" />
+      <mass value="2.46800319485063" />
       <inertia
         ixx="0.0218761505445032"
@@ -225,24 +156,17 @@
     </inertial>
     <visual>
-      <origin
-        xyz="0 0 0"
-        rpy="0 0 0" />
-      <geometry>
-        <mesh
-          filename="package://MarsRover/meshes/LeftMiddleWheel.STL" />
-      </geometry>
-      <material
-        name="">
-        <color
-          rgba="0.792156862745098 0.819607843137255 0.933333333333333 1" />
-      </material>
-    </visual>
-    <collision>
-      <origin
-        xyz="0 0 0"
-        rpy="0 0 0" />
-      <geometry>
-        <mesh
-          filename="package://MarsRover/meshes/LeftMiddleWheel.STL" />
+      <origin xyz="0 0 0" rpy="0 0 0" />
+      <geometry>
+        <mesh filename="package://mars_rover/meshes/LeftMiddleWheel.STL" />
+      </geometry>
+      <material name="">
+        <color rgba="0.792156862745098 0.819607843137255 0.933333333333333 1" />
+      </material>
+    </visual>
+    <collision>
+      <origin xyz="0 0 0" rpy="0 0 0" />
+      <geometry>
+        <mesh
+          filename="package://mars_rover/meshes/LeftMiddleWheel.STL" />
       </geometry>
     </collision>
@@ -283,5 +207,5 @@
       <geometry>
         <mesh
-          filename="package://MarsRover/meshes/LeftRearWheel.STL" />
+          filename="package://mars_rover/meshes/LeftRearWheel.STL" />
       </geometry>
       <material
@@ -297,5 +221,5 @@
       <geometry>
         <mesh
-          filename="package://MarsRover/meshes/LeftRearWheel.STL" />
+          filename="package://mars_rover/meshes/LeftRearWheel.STL" />
       </geometry>
     </collision>
@@ -336,5 +260,5 @@
       <geometry>
         <mesh
-          filename="package://MarsRover/meshes/LeftFrontWheel.STL" />
+          filename="package://mars_rover/meshes/LeftFrontWheel.STL" />
       </geometry>
       <material
@@ -350,5 +274,5 @@
       <geometry>
         <mesh
-          filename="package://MarsRover/meshes/LeftFrontWheel.STL" />
+          filename="package://mars_rover/meshes/LeftFrontWheel.STL" />
       </geometry>
     </collision>
@@ -367,57 +291,4 @@
       xyz="0 0 -1" />
   </joint>
-  <!--link
-    name="LeftDiffBarLink">
-    <inertial>
-      <origin
-        xyz="0.100844514587008 0 0"
-        rpy="0 0 0" />
-      <mass
-        value="0.200751056745894" />
-      <inertia
-        ixx="1.70941578635533E-05"
-        ixy="1.00926628658576E-19"
-        ixz="4.58491019961146E-19"
-        iyy="0.00141233412869607"
-        iyz="1.74566677143738E-10"
-        izz="0.00141233526669787" />
-    </inertial>
-    <visual>
-      <origin
-        xyz="0 0 0"
-        rpy="0 0 0" />
-      <geometry>
-        <mesh
-          filename="package://MarsRover/meshes/LeftDiffBarLink.STL" />
-      </geometry>
-      <material
-        name="">
-        <color
-          rgba="0.898039215686275 0.917647058823529 0.929411764705882 1" />
-      </material>
-    </visual>
-    <collision>
-      <origin
-        xyz="0 0 0"
-        rpy="0 0 0" />
-      <geometry>
-        <mesh
-          filename="package://MarsRover/meshes/LeftDiffBarLink.STL" />
-      </geometry>
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
File: urdf/PandarQT.xacro (robot description, xacro)
@@ -1,35 +1,10 @@
 <?xml version="1.0"?>
-<robot xmlns:xacro="http://www.ros.org/wiki/xacro" name="PandarQT">
+<robot xmlns:xacro="http://www.ros.org/wiki/xacro" name="PandarQT_LiDAR">
   <xacro:property name="PI" value="3.1415926535897931" />
-  <xacro:macro name="PandarQT" params="*origin parent:=base_link name:=velodyne topic:=PandarQT_Data hz:=10 lasers:=64 samples:=2187 min_range:=0.1 max_range:=30.0 min_angle_h:=-180 max_angle_h:=180 min_angle_v:=-52.1 max_angle_v:=52.1 resolution:=0.02 noise:=0.008 visual:=true gpu:=false">
-    <joint name="joint_${parent}_${name}" type="fixed">
-      <xacro:insert_block name="origin" />
-      <parent link="${parent}"/>
-      <child link="${name}_Link"/>
-    </joint>
-    <link name="${name}_Link">
-      <inertial>
-        <mass value="0.47584" />
-        <origin xyz="9.4172E-09 -0.012924 0.00012666" rpy="${PI/2} 0 0" />
-        <inertia ixx="0.00040186" ixy="1.5748E-10" ixz="-1.4024E-10"
-          iyy="0.0003397" iyz="1.3527E-06" izz="0.00040759" />
-      </inertial>
-      <visual>
-        <origin xyz="0 0 0" rpy="${PI/2} 0 0" />
-        <geometry>
-          <mesh filename="package://MarsRover/meshes/LiDAR.STL" />
-        </geometry>
-      </visual>
-      <collision>
-        <origin xyz="0 0 0" rpy="${PI/2} 0 0" />
-        <geometry>
-          <mesh filename="package://MarsRover/meshes/LiDAR.STL" />
-        </geometry>
-      </collision>
-    </link>
+  <xacro:macro name="PandarQT" params="link:=base_link topic:=PandarQT_Data hz:=10 lasers:=64 samples:=2187 min_range:=0.1 max_range:=30.0 min_angle_h:=-180 max_angle_h:=180 min_angle_v:=-52.1 max_angle_v:=52.1 resolution:=0.02 noise:=0.008 visual:=true gpu:=false">
     <!-- Gazebo requires the velodyne_gazebo_plugins package -->
-    <gazebo reference="${name}_Link">
+    <gazebo reference="${link}">
       <xacro:if value="${gpu}">
-        <sensor type="gpu_ray" name="${name}_Sensor">
+        <sensor type="gpu_ray" name="${link}_Sensor">
           <pose>0 0 0 0 0 0</pose>
           <visualize>${visual}</visualize>
@@ -67,15 +42,16 @@
             </noise>
           </ray>
-          <plugin name="gazebo_ros_laser_controller" filename="$(find MarsRover)/plugins/LidarPubData/build/libLidarPubData.so">
+          <plugin name="LidarPubData" filename="$(find mars_rover)/plugins/LidarPubData/build/libLidarPubData.so">
             <topicName>${topic}</topicName>
-            <frameName>${name}</frameName>
+            <frameName>${link}</frameName>
             <min_range>${min_range}</min_range>
             <max_range>${max_range}</max_range>
             <gaussianNoise>${noise}</gaussianNoise>
+            <min_intensity>0</min_intensity>
           </plugin>
         </sensor>
       </xacro:if>
       <xacro:unless value="${gpu}">
-        <sensor type="ray" name="${name}-HDL32E">
+        <sensor type="ray" name="${link}_Sensor">
           <pose>0 0 0 0 0 0</pose>
           <visualize>${visual}</visualize>
@@ -113,10 +89,11 @@
             </noise>
           </ray>
-          <plugin name="gazebo_ros_laser_controller" filename="$(find MarsRover)/plugins/LidarPubData/build/libLidarPubData.so">
+          <plugin name="LidarPubData" filename="$(find mars_rover)/plugins/LidarPubData/build/libLidarPubData.so">
             <topicName>${topic}</topicName>
-            <frameName>${name}</frameName>
+            <frameName>${link}</frameName>
             <min_range>${min_range}</min_range>
             <max_range>${max_range}</max_range>
             <gaussianNoise>${noise}</gaussianNoise>
+            <min_intensity>0</min_intensity>
           </plugin>
         </sensor>
