Commit message: 修改部分标签的格式以及值，删除部分不需要的标签

File: urdf/MarsRover.xacro (robot description, xacro)
@@ -12,5 +12,5 @@
   <link name="body">
     <inertial>
-      <origin xyz="-0.000147897244928197 -0.0822271126898096 1.11022302462516E-16" rpy="0 0 0" />
+      <origin xyz="-0.000147897244928197 -0.0822271126898096 0" rpy="0 0 0" />
       <mass value="32.9286570826472" />
       <inertia
@@ -41,5 +41,5 @@
     name="DiffBar">
     <inertial>
-      <origin xyz="7.23369697475107E-10 -0.0223125966605722 3.3729640969149E-08" rpy="0 0 0" />
+      <origin xyz="0 -0.0223125966605722 0" rpy="0 0 0" />
       <mass value="1.49170112220708" />
       <inertia
@@ -145,5 +145,5 @@
   <link name="LeftMiddleWheel">
     <inertial>
-      <origin xyz="0 -2.77555756156289E-17 1.66533453693773E-16" rpy="0 0 0" />
+      <origin xyz="0 0 0" rpy="0 0 0" />
       <mass value="2.46800319485063" />
       <inertia
@@ -167,30 +167,18 @@
       <origin xyz="0 0 0" rpy="0 0 0" />
       <geometry>
-        <mesh
-          filename="package://mars_rover/meshes/LeftMiddleWheel.STL" />
-      </geometry>
-    </collision>
-  </link>
-  <joint
-    name="joint_LeftViceRocker_LeftMiddleWheel"
-    type="continuous">
-    <origin
-      xyz="0.38804 -0.24313 -0.09"
-      rpy="0 0 0" />
-    <parent
-      link="LeftViceRocker" />
-    <child
-      link="LeftMiddleWheel" />
-    <axis
-      xyz="0 0 -1" />
-  </joint>
-  <link
-    name="LeftRearWheel">
-    <inertial>
-      <origin
-        xyz="-5.55111512312578E-17 0 5.55111512312578E-17"
-        rpy="0 0 0" />
-      <mass
-        value="2.46800319485063" />
+        <mesh filename="package://mars_rover/meshes/LeftMiddleWheel.STL" />
+      </geometry>
+    </collision>
+  </link>
+  <joint name="joint_LeftViceRocker_LeftMiddleWheel" type="continuous">
+    <origin xyz="0.38804 -0.24313 -0.09" rpy="0 0 0" />
+    <parent link="LeftViceRocker" />
+    <child link="LeftMiddleWheel" />
+    <axis xyz="0 0 -1" />
+  </joint>
+  <link name="LeftRearWheel">
+    <inertial>
+      <origin xyz="0 0 0" rpy="0 0 0" />
+      <mass value="2.46800319485063" />
       <inertia
         ixx="0.0218761505445031"
@@ -202,48 +190,29 @@
     </inertial>
     <visual>
-      <origin
-        xyz="0 0 0"
-        rpy="0 0 0" />
-      <geometry>
-        <mesh
-          filename="package://mars_rover/meshes/LeftRearWheel.STL" />
-      </geometry>
-      <material
-        name="">
-        <color
-          rgba="0.792156862745098 0.819607843137255 0.933333333333333 1" />
-      </material>
-    </visual>
-    <collision>
-      <origin
-        xyz="0 0 0"
-        rpy="0 0 0" />
-      <geometry>
-        <mesh
-          filename="package://mars_rover/meshes/LeftRearWheel.STL" />
-      </geometry>
-    </collision>
-  </link>
-  <joint
-    name="joint_LeftViceRocker_LeftRearWheel"
-    type="continuous">
-    <origin
-      xyz="-0.38693 -0.2449 -0.09"
-      rpy="0 0 0" />
-    <parent
-      link="LeftViceRocker" />
-    <child
-      link="LeftRearWheel" />
-    <axis
-      xyz="0 0 -1" />
-  </joint>
-  <link
-    name="LeftFrontWheel">
-    <inertial>
-      <origin
-        xyz="0 8.32667268468867E-17 0"
-        rpy="0 0 0" />
-      <mass
-        value="2.46800319485063" />
+      <origin xyz="0 0 0" rpy="0 0 0" />
+      <geometry>
+        <mesh filename="package://mars_rover/meshes/LeftRearWheel.STL" />
+      </geometry>
+      <material name="">
+        <color rgba="0.792156862745098 0.819607843137255 0.933333333333333 1" />
+      </material>
+    </visual>
+    <collision>
+      <origin xyz="0 0 0" rpy="0 0 0" />
+      <geometry>
+        <mesh filename="package://mars_rover/meshes/LeftRearWheel.STL" />
+      </geometry>
+    </collision>
+  </link>
+  <joint name="joint_LeftViceRocker_LeftRearWheel" type="continuous">
+    <origin xyz="-0.38693 -0.2449 -0.09" rpy="0 0 0" />
+    <parent link="LeftViceRocker" />
+    <child link="LeftRearWheel" />
+    <axis xyz="0 0 -1" />
+  </joint>
+  <link name="LeftFrontWheel">
+    <inertial>
+      <origin xyz="0 0 0" rpy="0 0 0" />
+      <mass value="2.46800319485063" />
       <inertia
         ixx="0.0218761505445031"
@@ -255,48 +224,29 @@
     </inertial>
     <visual>
-      <origin
-        xyz="0 0 0"
-        rpy="0 0 0" />
-      <geometry>
-        <mesh
-          filename="package://mars_rover/meshes/LeftFrontWheel.STL" />
-      </geometry>
-      <material
-        name="">
-        <color
-          rgba="0.792156862745098 0.819607843137255 0.933333333333333 1" />
-      </material>
-    </visual>
-    <collision>
-      <origin
-        xyz="0 0 0"
-        rpy="0 0 0" />
-      <geometry>
-        <mesh
-          filename="package://mars_rover/meshes/LeftFrontWheel.STL" />
-      </geometry>
-    </collision>
-  </link>
-  <joint
-    name="joint_LeftMainRocker_LeftFrontWheel"
-    type="continuous">
-    <origin
-      xyz="0.75893 -0.27932 -0.145"
-      rpy="0 0 0" />
-    <parent
-      link="LeftMainRocker" />
-    <child
-      link="LeftFrontWheel" />
-    <axis
-      xyz="0 0 -1" />
-  </joint>
-  <link
-    name="RightMainRocker">
-    <inertial>
-      <origin
-        xyz="0.194763676146297 -0.101665854830299 0.0322193239500774"
-        rpy="0 0 0" />
-      <mass
-        value="2.31657690221752" />
+      <origin xyz="0 0 0" rpy="0 0 0" />
+      <geometry>
+        <mesh filename="package://mars_rover/meshes/LeftFrontWheel.STL" />
+      </geometry>
+      <material name="">
+        <color rgba="0.792156862745098 0.819607843137255 0.933333333333333 1" />
+      </material>
+    </visual>
+    <collision>
+      <origin xyz="0 0 0" rpy="0 0 0" />
+      <geometry>
+        <mesh filename="package://mars_rover/meshes/LeftFrontWheel.STL" />
+      </geometry>
+    </collision>
+  </link>
+  <joint name="joint_LeftMainRocker_LeftFrontWheel" type="continuous">
+    <origin xyz="0.75893 -0.27932 -0.145" rpy="0 0 0" />
+    <parent link="LeftMainRocker" />
+    <child link="LeftFrontWheel" />
+    <axis xyz="0 0 -1" />
+  </joint>
+  <link name="RightMainRocker">
+    <inertial>
+      <origin xyz="0.194763676146297 -0.101665854830299 0.0322193239500774" rpy="0 0 0" />
+      <mass value="2.31657690221752" />
       <inertia
         ixx="0.0253400528535679"
@@ -308,48 +258,29 @@
     </inertial>
     <visual>
-      <origin
-        xyz="0 0 0"
-        rpy="0 0 0" />
-      <geometry>
-        <mesh
-          filename="package://mars_rover/meshes/RightMainRocker.STL" />
-      </geometry>
-      <material
-        name="">
-        <color
-          rgba="0.792156862745098 0.819607843137255 0.933333333333333 1" />
-      </material>
-    </visual>
-    <collision>
-      <origin
-        xyz="0 0 0"
-        rpy="0 0 0" />
-      <geometry>
-        <mesh
-          filename="package://mars_rover/meshes/RightMainRocker.STL" />
-      </geometry>
-    </collision>
-  </link>
-  <joint
-    name="joint_body_RightMainRocker"
-    type="continuous">
-    <origin
-      xyz="0 -0.155 0.395"
-      rpy="0 0 0" />
-    <parent
-      link="body" />
-    <child
-      link="RightMainRocker" />
-    <axis
-      xyz="0 0 1" />
-  </joint>
-  <link
-    name="RightViceRocker">
-    <inertial>
-      <origin
-        xyz="-3.74727935245119E-05 -0.142829300218082 0.00457781208829156"
-        rpy="0 0 0" />
-      <mass
-        value="1.70193743881046" />
+      <origin xyz="0 0 0" rpy="0 0 0" />
+      <geometry>
+        <mesh filename="package://mars_rover/meshes/RightMainRocker.STL" />
+      </geometry>
+      <material name="">
+        <color rgba="0.792156862745098 0.819607843137255 0.933333333333333 1" />
+      </material>
+    </visual>
+    <collision>
+      <origin xyz="0 0 0" rpy="0 0 0" />
+      <geometry>
+        <mesh filename="package://mars_rover/meshes/RightMainRocker.STL" />
+      </geometry>
+    </collision>
+  </link>
+  <joint name="joint_body_RightMainRocker" type="continuous">
+    <origin xyz="0 -0.155 0.395" rpy="0 0 0" />
+    <parent link="body" />
+    <child link="RightMainRocker" />
+    <axis xyz="0 0 1" />
+  </joint>
+  <link name="RightViceRocker">
+    <inertial>
+      <origin xyz="0 -0.142829300218082 0.00457781208829156" rpy="0 0 0" />
+      <mass value="1.70193743881046" />
       <inertia
         ixx="0.0116402353185612"
@@ -361,48 +292,29 @@
     </inertial>
     <visual>
-      <origin
-        xyz="0 0 0"
-        rpy="0 0 0" />
-      <geometry>
-        <mesh
-          filename="package://mars_rover/meshes/RightViceRocker.STL" />
-      </geometry>
-      <material
-        name="">
-        <color
-          rgba="0.792156862745098 0.819607843137255 0.933333333333333 1" />
-      </material>
-    </visual>
-    <collision>
-      <origin
-        xyz="0 0 0"
-        rpy="0 0 0" />
-      <geometry>
-        <mesh
-          filename="package://mars_rover/meshes/RightViceRocker.STL" />
-      </geometry>
-    </collision>
-  </link>
-  <joint
-    name="joint_RightMainRocker_RightViceRocker"
-    type="continuous">
-    <origin
-      xyz="-0.40088 -0.023015 0.055"
-      rpy="0 0 0" />
-    <parent
-      link="RightMainRocker" />
-    <child
-      link="RightViceRocker" />
-    <axis
-      xyz="0 0 1" />
-  </joint>
-  <link
-    name="RightMiddleWheel">
-    <inertial>
-      <origin
-        xyz="5.55111512312578E-17 2.77555756156289E-17 4.44089209850063E-16"
-        rpy="0 0 0" />
-      <mass
-        value="2.46800319485063" />
+      <origin xyz="0 0 0" rpy="0 0 0" />
+      <geometry>
+        <mesh filename="package://mars_rover/meshes/RightViceRocker.STL" />
+      </geometry>
+      <material name="">
+        <color rgba="0.792156862745098 0.819607843137255 0.933333333333333 1" />
+      </material>
+    </visual>
+    <collision>
+      <origin xyz="0 0 0" rpy="0 0 0" />
+      <geometry>
+        <mesh filename="package://mars_rover/meshes/RightViceRocker.STL" />
+      </geometry>
+    </collision>
+  </link>
+  <joint name="joint_RightMainRocker_RightViceRocker" type="continuous">
+    <origin xyz="-0.40088 -0.023015 0.055" rpy="0 0 0" />
+    <parent link="RightMainRocker" />
+    <child link="RightViceRocker" />
+    <axis xyz="0 0 1" />
+  </joint>
+  <link name="RightMiddleWheel">
+    <inertial>
+      <origin xyz="0 0 0" rpy="0 0 0" />
+      <mass value="2.46800319485063" />
       <inertia
         ixx="0.0218761505445029"
@@ -414,48 +326,29 @@
     </inertial>
     <visual>
-      <origin
-        xyz="0 0 0"
-        rpy="0 0 0" />
-      <geometry>
-        <mesh
-          filename="package://mars_rover/meshes/RightMiddleWheel.STL" />
-      </geometry>
-      <material
-        name="">
-        <color
-          rgba="0.792156862745098 0.819607843137255 0.933333333333333 1" />
-      </material>
-    </visual>
-    <collision>
-      <origin
-        xyz="0 0 0"
-        rpy="0 0 0" />
-      <geometry>
-        <mesh
-          filename="package://mars_rover/meshes/RightMiddleWheel.STL" />
-      </geometry>
-    </collision>
-  </link>
-  <joint
-    name="joint_RightViceRocker_RightMiddleWheel"
-    type="continuous">
-    <origin
-      xyz="0.38742 -0.24412 0.09"
-      rpy="0 0 0" />
-    <parent
-      link="RightViceRocker" />
-    <child
-      link="RightMiddleWheel" />
-    <axis
-      xyz="0 0 1" />
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
Commit message: 1.不使用rviz显示点云图像，调用ros和pcl库编写接收、显示点云数据的程序并在launch文件中启动该程序节点； 2.由于键盘只能控制小车前进后退转弯，无法控制速度，因此在处理键盘输入的程序中添加了实时获取ros参数服务器中小车速度设定相关参数的功能。

File: urdf/MarsRover.xacro (robot description, xacro)
@@ -10,4 +10,9 @@
   <xacro:property name="LidarHeight" value="-0.0" />
   <xacro:property name="LidarName" value="PandarQT" />
+  <xacro:property name="LidarDataTopicName" value="PandarQT_Data" />
+  <xacro:property name="LidarHz" value="10" />
+  <xacro:property name="LidarLasers" value="64" />
+  <xacro:property name="LidarSamples" value="600" />
+  <xacro:property name="LidarBeamVisual" value="false" />
   <link name="body">
     <inertial>
@@ -342,5 +347,5 @@
   </link>
   <joint name="joint_RightViceRocker_RightMiddleWheel" type="continuous">
-    <origin xyz="0.38742 -0.24412 0.09" rpy="0 0 0" />
+    <origin xyz="0.38742 -0.24412 0.09" rpy="${PI} 0 0" />
     <parent link="RightViceRocker" />
     <child link="RightMiddleWheel" />
@@ -376,5 +381,5 @@
   </link>
   <joint name="joint_RightViceRocker_RightRearWheel" type="continuous">
-    <origin xyz="-0.38755 -0.24391 0.09" rpy="0 0 0" />
+    <origin xyz="-0.38755 -0.24391 0.09" rpy="${PI} 0 0" />
     <parent link="RightViceRocker" />
     <child link="RightRearWheel" />
@@ -410,5 +415,5 @@
   </link>
   <joint name="joint_RightMainRocker_RightFrontWheel" type="continuous">
-    <origin xyz="0.75889 -0.27943 0.145" rpy="0 0 0" />
+    <origin xyz="0.75889 -0.27943 0.145" rpy="${PI} 0 0" />
     <parent link="RightMainRocker" />
     <child link="RightFrontWheel" />
@@ -520,4 +525,4 @@
     </joint>
     <xacro:include filename="$(find mars_rover)/urdf/PandarQT.xacro"/>
-    <xacro:PandarQT link="${LidarName}" topic="PandarQT_Data" hz="10" lasers="64" samples="600" visual="false"></xacro:PandarQT>
+    <xacro:PandarQT link="${LidarName}" topic="${LidarDataTopicName}" hz="${LidarHz}" lasers="${LidarLasers}" samples="${LidarSamples}" visual="${LidarBeamVisual}"></xacro:PandarQT>
 </robot>

Commit message: 在Gazebo中添加了IMU传感器，并将插件程序在本地进行了编译； 在获取激光雷达仿真数据的插件程序中修改了输出的PointCloud2点云的点的格式，使之与禾赛PandarQT输出点云的点的格式一致； 在获取激光雷达仿真数据的插件程序中添加了剔除指定水平方位角和线束范围内的点的功能。

File: urdf/MarsRover.xacro (robot description, xacro)
@@ -524,5 +524,6 @@
       <child link="${LidarName}"/>
     </joint>
-    <xacro:include filename="$(find mars_rover)/urdf/PandarQT.xacro"/>
+    <xacro:include filename="$(find mars_rover)/urdf/Sensors.xacro"/>
     <xacro:PandarQT link="${LidarName}" topic="${LidarDataTopicName}" hz="${LidarHz}" lasers="${LidarLasers}" samples="${LidarSamples}" visual="${LidarBeamVisual}"></xacro:PandarQT>
+    <xacro:IMU link="${LidarName}" pitch="${0}" gaussianNoise="0.0"></xacro:IMU>
 </robot>

File: urdf/Sensors.xacro (robot description, xacro)
@@ -2,5 +2,5 @@
 <robot xmlns:xacro="http://www.ros.org/wiki/xacro" name="PandarQT_LiDAR">
   <xacro:property name="PI" value="3.1415926535897931" />
-  <xacro:macro name="PandarQT" params="link:=base_link topic:=PandarQT_Data hz:=10 lasers:=64 samples:=2187 min_range:=0.1 max_range:=30.0 min_angle_h:=-180 max_angle_h:=180 min_angle_v:=-52.1 max_angle_v:=52.1 resolution:=0.02 noise:=0.008 visual:=true gpu:=false">
+  <xacro:macro name="PandarQT" params="link:=base_link topic:=PandarQT_Data hz:=10 lasers:=64 samples:=2187 min_range:=0.8 max_range:=30.0 min_angle_h:=-180 max_angle_h:=180 min_angle_v:=-52.1 max_angle_v:=52.1 resolution:=0.02 noise:=0.008 visual:=true gpu:=false">
     <!-- Gazebo requires the velodyne_gazebo_plugins package -->
     <gazebo reference="${link}">
@@ -42,4 +42,5 @@
             </noise>
           </ray>
+          <!--该角度以绕Z轴由X轴转至Y轴为正方向，X轴正方向为起始，Gazebo仿真里面Lidar的角度以X轴负方向为起始 -->
           <plugin name="LidarPubData" filename="$(find mars_rover)/plugins/LidarPubData/build/libLidarPubData.so">
             <topicName>${topic}</topicName>
@@ -49,4 +50,8 @@
             <gaussianNoise>${noise}</gaussianNoise>
             <min_intensity>0</min_intensity>
+            <ignoreAzimuthAngleUp>240</ignoreAzimuthAngleUp>
+            <ignoreAzimuthAngleLow>120</ignoreAzimuthAngleLow>
+            <ignoreScanIDUp>44</ignoreScanIDUp>
+            <ignoreScanIDLow>6</ignoreScanIDLow>
           </plugin>
         </sensor>
@@ -89,5 +94,5 @@
             </noise>
           </ray>
-          <plugin name="LidarPubData" filename="$(find mars_rover)/plugins/LidarPubData/build/libLidarPubData.so">
+          <plugin name="LidarPubData" filename="$(find mars_rover)/plugins/LidarPubData/build/libLidarPubData_plugins.so">
             <topicName>${topic}</topicName>
             <frameName>${link}</frameName>
@@ -96,4 +101,8 @@
             <gaussianNoise>${noise}</gaussianNoise>
             <min_intensity>0</min_intensity>
+            <ignoreAzimuthAngleUp>320</ignoreAzimuthAngleUp>
+            <ignoreAzimuthAngleLow>40</ignoreAzimuthAngleLow>
+            <ignoreScanIDUp>44</ignoreScanIDUp>
+            <ignoreScanIDLow>12</ignoreScanIDLow>
           </plugin>
         </sensor>
@@ -101,3 +110,24 @@
     </gazebo>
   </xacro:macro>
+  <xacro:macro name="IMU" params="link:=base_link enable_gravity:=true imu_name:=imu_1 hz:=100 enable_visual:=true topic_name:=imu_raw frameName:=imu_link gaussianNoise:=0.1 x:=0 y:=0 z:=0 roll:=0 pitch:=0 yaw:=0">
+    <gazebo reference="${link}">
+      <gravity>${enable_gravity}</gravity>
+      <sensor name="${imu_name}" type="imu">
+        <always_on>true</always_on>
+        <update_rate>${hz}</update_rate>
+        <visualize>${enable_visual}</visualize>
+        <topic>${topic_name}</topic>
+        <plugin name="imu_plugin" filename="$(find mars_rover)/plugins/ImuPubData/build/libImuPubData_plugins.so">
+          <topicName>${topic_name}</topicName>
+          <bodyName>${link}</bodyName>
+          <updateRateHZ>${hz}</updateRateHZ>
+          <gaussianNoise>${gaussianNoise}</gaussianNoise>
+          <xyzOffset>${x} ${y} ${z}</xyzOffset>
+          <rpyOffset>${roll} ${pitch} ${yaw}</rpyOffset>
+          <frameName>${link}</frameName>
+        </plugin>
+        <pose>0 0 0 0 0 0</pose>
+      </sensor>
+    </gazebo>
+  </xacro:macro>
 </robot>

Commit message: 。。。

File: urdf/MarsRover.xacro (robot description, xacro)
@@ -7,5 +7,5 @@
   <xacro:include filename="$(find mars_rover)/urdf/MarsRover.gazebo" />
   <xacro:property name="PI" value="3.141592654" />
-  <xacro:property name="LidarAngle" value="${PI/6}" />
+  <xacro:property name="LidarAngle" value="${PI/180*65}" />
   <xacro:property name="LidarHeight" value="-0.0" />
   <xacro:property name="LidarName" value="PandarQT" />

File: urdf/Sensors.xacro (robot description, xacro)
@@ -2,5 +2,5 @@
 <robot xmlns:xacro="http://www.ros.org/wiki/xacro" name="PandarQT_LiDAR">
   <xacro:property name="PI" value="3.1415926535897931" />
-  <xacro:macro name="PandarQT" params="link:=base_link topic:=PandarQT_Data hz:=10 lasers:=64 samples:=2187 min_range:=0.8 max_range:=30.0 min_angle_h:=-180 max_angle_h:=180 min_angle_v:=-52.1 max_angle_v:=52.1 resolution:=0.02 noise:=0.008 visual:=true gpu:=false">
+  <xacro:macro name="PandarQT" params="link:=base_link topic:=PandarQT_Data hz:=10 lasers:=64 samples:=2187 min_range:=0.8 max_range:=30.0 min_angle_h:=-180 max_angle_h:=180 min_angle_v:=-52.1 max_angle_v:=52.1 resolution:=0.02 noise:=0.00 visual:=true gpu:=false">
     <!-- Gazebo requires the velodyne_gazebo_plugins package -->
     <gazebo reference="${link}">
@@ -43,5 +43,5 @@
           </ray>
           <!--该角度以绕Z轴由X轴转至Y轴为正方向，X轴正方向为起始，Gazebo仿真里面Lidar的角度以X轴负方向为起始 -->
-          <plugin name="LidarPubData" filename="$(find mars_rover)/plugins/LidarPubData/build/libLidarPubData.so">
+          <plugin name="LidarPubData" filename="$(find mars_rover)/plugins/LidarPubData/build/libLidarPubData_plugins.so">
             <topicName>${topic}</topicName>
             <frameName>${link}</frameName>
@@ -91,5 +91,5 @@
               <type>gaussian</type>
               <mean>0.0</mean>
-              <stddev>0.0</stddev>
+              <stddev>0.01</stddev>
             </noise>
           </ray>
@@ -101,8 +101,8 @@
             <gaussianNoise>${noise}</gaussianNoise>
             <min_intensity>0</min_intensity>
-            <ignoreAzimuthAngleUp>320</ignoreAzimuthAngleUp>
-            <ignoreAzimuthAngleLow>40</ignoreAzimuthAngleLow>
-            <ignoreScanIDUp>44</ignoreScanIDUp>
-            <ignoreScanIDLow>12</ignoreScanIDLow>
+            <ignoreAzimuthAngleUp>0.7</ignoreAzimuthAngleUp>
+            <ignoreAzimuthAngleLow>-0.7</ignoreAzimuthAngleLow>
+            <ignoreScanIDUp>27</ignoreScanIDUp>
+            <ignoreScanIDLow>-1</ignoreScanIDLow>
           </plugin>
         </sensor>

Commit message: 坐标系的设定有些问题，准备进行修改。

File: urdf/MarsRover.xacro (robot description, xacro)
@@ -30,5 +30,5 @@
       <origin xyz="0 0 0" rpy="0 0 0" />
       <geometry>
-        <mesh filename="package://mars_rover/meshes/body.STL" />
+        <mesh filename="package://mars_rover/meshes/body.dae" />
       </geometry>
       <material name="">
@@ -39,5 +39,5 @@
       <origin xyz="0 0 0" rpy="0 0 0" />
       <geometry>
-        <mesh filename="package://mars_rover/meshes/body.STL" />
+        <mesh filename="package://mars_rover/meshes/body.dae" />
       </geometry>
     </collision>
