Commit message: 完成了坐标系的修改，确保每一个link的坐标系都是X轴朝前，Y轴朝左，Z轴朝上；同时每个link的模型采用了dae文件，使用Blender为原始的STL文件上色并输出为dae文件。

File: urdf/MarsRover.xacro (robot description, xacro)
@@ -7,5 +7,5 @@
   <xacro:include filename="$(find mars_rover)/urdf/MarsRover.gazebo" />
   <xacro:property name="PI" value="3.141592654" />
-  <xacro:property name="LidarAngle" value="${PI/180*65}" />
+  <xacro:property name="LidarAngle" value="${PI/180*0}" />
   <xacro:property name="LidarHeight" value="-0.0" />
   <xacro:property name="LidarName" value="PandarQT" />
@@ -15,29 +15,41 @@
   <xacro:property name="LidarSamples" value="600" />
   <xacro:property name="LidarBeamVisual" value="false" />
-  <link name="body">
-    <inertial>
-      <origin xyz="-0.000147897244928197 -0.0822271126898096 0" rpy="0 0 0" />
-      <mass value="32.9286570826472" />
-      <inertia
-        ixx="4.47491142188154"
-        ixy="-0.000503480655802534"
-        ixz="1.31725686550942E-14"
-        iyy="9.29423854790981"
-        iyz="7.44971011585177E-16"
-        izz="7.39741952054995" />
-    </inertial>
-    <visual>
-      <origin xyz="0 0 0" rpy="0 0 0" />
-      <geometry>
-        <mesh filename="package://mars_rover/meshes/body.dae" />
-      </geometry>
-      <material name="">
-        <color rgba="0.752941176470588 0.752941176470588 0.752941176470588 1" />
-      </material>
-    </visual>
-    <collision>
-      <origin xyz="0 0 0" rpy="0 0 0" />
-      <geometry>
-        <mesh filename="package://mars_rover/meshes/body.dae" />
+  <link
+    name="body">
+    <inertial>
+      <origin
+        xyz="-0.0001479 -1.1102E-16 -0.38223"
+        rpy="0 0 0" />
+      <mass
+        value="32.929" />
+      <inertia
+        ixx="4.4749"
+        ixy="-1.3173E-14"
+        ixz="-0.00050348"
+        iyy="7.3974"
+        iyz="-8.0126E-16"
+        izz="9.2942" />
+    </inertial>
+    <visual>
+      <origin
+        xyz="0 0 0"
+        rpy="0 0 0" />
+      <geometry>
+        <mesh
+          filename="package://mars_rover/meshes/body.dae" />
+      </geometry>
+      <material
+        name="">
+        <color
+          rgba="0.75294 0.75294 0.75294 1" />
+      </material>
+    </visual>
+    <collision>
+      <origin
+        xyz="0 0 0"
+        rpy="0 0 0" />
+      <geometry>
+        <mesh
+          filename="package://mars_rover/meshes/body.dae" />
       </geometry>
     </collision>
@@ -46,482 +58,854 @@
     name="DiffBar">
     <inertial>
-      <origin xyz="0 -0.0223125966605722 0" rpy="0 0 0" />
-      <mass value="1.49170112220708" />
-      <inertia
-        ixx="0.030385701616174"
-        ixy="-4.27358554206539E-11"
-        ixz="6.00528612798054E-07"
-        iyy="0.0300953010528317"
-        iyz="1.87976912025262E-08"
-        izz="0.000583955549724061" />
-    </inertial>
-    <visual>
-      <origin xyz="0 0 0" rpy="0 0 0" />
-      <geometry>
-        <mesh filename="package://mars_rover/meshes/DiffBar.STL" />
-      </geometry>
-      <material name="">
-        <color rgba="0.898039215686275 0.917647058823529 0.929411764705882 1" />
-      </material>
-    </visual>
-    <collision>
-      <origin xyz="0 0 0" rpy="0 0 0" />
-      <geometry>
-        <mesh filename="package://mars_rover/meshes/DiffBar.STL" />
-      </geometry>
-    </collision>
-  </link>
-  <joint name="joint_body_DiffBar" type="continuous">
-    <origin xyz="0.20043 -0.225 0" rpy="0 0 0" />
-    <parent link="body" />
-    <child link="DiffBar" />
-    <axis xyz="0 1 0" />
-  </joint>
-  <link name="LeftMainRocker">
-    <inertial>
-      <origin xyz="0.194777234245267 -0.101638011239522 -0.0322190943393932" rpy="0 0 0" />
-      <mass value="2.31659033764537" />
-      <inertia
-        ixx="0.0253182901443958"
-        ixy="0.0763954336660846"
-        ixz="0.00562994284708994"
-        iyy="0.301511476413955"
-        iyz="-0.00212772758361841"
-        izz="0.322973812666095" />
-    </inertial>
-    <visual>
-      <origin xyz="0 0 0" rpy="0 0 0" />
-      <geometry>
-        <mesh filename="package://mars_rover/meshes/LeftMainRocker.STL" />
-      </geometry>
-      <material name="">
-        <color rgba="0.792156862745098 0.819607843137255 0.933333333333333 1" />
-      </material>
-    </visual>
-    <collision>
-      <origin xyz="0 0 0" rpy="0 0 0" />
-      <geometry>
-        <mesh filename="package://mars_rover/meshes/LeftMainRocker.STL" />
-      </geometry>
-    </collision>
-  </link>
-  <joint name="joint_body_LeftMainRocker" type="continuous">
-    <origin xyz="0 -0.155 -0.395" rpy="0 0 0" />
-    <parent link="body" />
-    <child link="LeftMainRocker" />
-    <axis xyz="0 0 1" />
-  </joint>
-  <link name="LeftViceRocker">
-    <inertial>
-      <origin
-        xyz="0.000324935586217618 -0.142828935520301 -0.00457781208829167"
-        rpy="0 0 0" />
-      <mass value="1.70193743881046" />
-      <inertia
-        ixx="0.011640762472159"
-        ixy="-0.000234839301434703"
-        ixz="1.79349163947906E-06"
-        iyy="0.114866371685707"
-        iyz="-0.000788348560750385"
-        izz="0.1254823143192" />
-    </inertial>
-    <visual>
-      <origin xyz="0 0 0" rpy="0 0 0" />
-      <geometry>
-        <mesh filename="package://mars_rover/meshes/LeftViceRocker.STL" />
-      </geometry>
-      <material name="">
-        <color rgba="0.792156862745098 0.819607843137255 0.933333333333333 1" />
-      </material>
-    </visual>
-    <collision>
-      <origin xyz="0 0 0" rpy="0 0 0" />
-      <geometry>
-        <mesh filename="package://mars_rover/meshes/LeftViceRocker.STL" />
-      </geometry>
-    </collision>
-  </link>
-  <joint name="joint_LeftMainRocker_LeftViceRocker" type="continuous">
-    <origin xyz="-0.40088 -0.023072 -0.055" rpy="0 0 0" />
-    <parent link="LeftMainRocker" />
-    <child link="LeftViceRocker" />
-    <axis xyz="0 0 1" />
-  </joint>
-  <link name="LeftMiddleWheel">
-    <inertial>
-      <origin xyz="0 0 0" rpy="0 0 0" />
-      <mass value="2.46800319485063" />
-      <inertia
-        ixx="0.0218761505445032"
-        ixy="-1.19260452263282E-17"
-        ixz="-8.56630017307201E-19"
-        iyy="0.0218761505445032"
-        iyz="4.7148329734938E-18"
-        izz="0.0405258063947127" />
-    </inertial>
-    <visual>
-      <origin xyz="0 0 0" rpy="0 0 0" />
-      <geometry>
-        <mesh filename="package://mars_rover/meshes/LeftMiddleWheel.STL" />
-      </geometry>
-      <material name="">
-        <color rgba="0.792156862745098 0.819607843137255 0.933333333333333 1" />
-      </material>
-    </visual>
-    <collision>
-      <origin xyz="0 0 0" rpy="0 0 0" />
-      <geometry>
-        <mesh filename="package://mars_rover/meshes/LeftMiddleWheel.STL" />
-      </geometry>
-    </collision>
-  </link>
-  <joint name="joint_LeftViceRocker_LeftMiddleWheel" type="continuous">
-    <origin xyz="0.38804 -0.24313 -0.09" rpy="0 0 0" />
-    <parent link="LeftViceRocker" />
-    <child link="LeftMiddleWheel" />
-    <axis xyz="0 0 -1" />
-  </joint>
-  <link name="LeftRearWheel">
-    <inertial>
-      <origin xyz="0 0 0" rpy="0 0 0" />
-      <mass value="2.46800319485063" />
-      <inertia
-        ixx="0.0218761505445031"
-        ixy="-1.52170599454406E-17"
-        ixz="-1.27014873364989E-18"
-        iyy="0.0218761505445032"
-        iyz="1.03685045793585E-19"
-        izz="0.040525806394713" />
-    </inertial>
-    <visual>
-      <origin xyz="0 0 0" rpy="0 0 0" />
-      <geometry>
-        <mesh filename="package://mars_rover/meshes/LeftRearWheel.STL" />
-      </geometry>
-      <material name="">
-        <color rgba="0.792156862745098 0.819607843137255 0.933333333333333 1" />
-      </material>
-    </visual>
-    <collision>
-      <origin xyz="0 0 0" rpy="0 0 0" />
-      <geometry>
-        <mesh filename="package://mars_rover/meshes/LeftRearWheel.STL" />
-      </geometry>
-    </collision>
-  </link>
-  <joint name="joint_LeftViceRocker_LeftRearWheel" type="continuous">
-    <origin xyz="-0.38693 -0.2449 -0.09" rpy="0 0 0" />
-    <parent link="LeftViceRocker" />
-    <child link="LeftRearWheel" />
-    <axis xyz="0 0 -1" />
-  </joint>
-  <link name="LeftFrontWheel">
-    <inertial>
-      <origin xyz="0 0 0" rpy="0 0 0" />
-      <mass value="2.46800319485063" />
-      <inertia
-        ixx="0.0218761505445031"
-        ixy="1.11983361154303E-17"
-        ixz="1.57073225640767E-18"
-        iyy="0.0218761505445032"
-        iyz="1.17261152392734E-18"
-        izz="0.0405258063947128" />
-    </inertial>
-    <visual>
-      <origin xyz="0 0 0" rpy="0 0 0" />
-      <geometry>
-        <mesh filename="package://mars_rover/meshes/LeftFrontWheel.STL" />
-      </geometry>
-      <material name="">
-        <color rgba="0.792156862745098 0.819607843137255 0.933333333333333 1" />
-      </material>
-    </visual>
-    <collision>
-      <origin xyz="0 0 0" rpy="0 0 0" />
-      <geometry>
-        <mesh filename="package://mars_rover/meshes/LeftFrontWheel.STL" />
-      </geometry>
-    </collision>
-  </link>
-  <joint name="joint_LeftMainRocker_LeftFrontWheel" type="continuous">
-    <origin xyz="0.75893 -0.27932 -0.145" rpy="0 0 0" />
-    <parent link="LeftMainRocker" />
-    <child link="LeftFrontWheel" />
-    <axis xyz="0 0 -1" />
-  </joint>
-  <link name="RightMainRocker">
-    <inertial>
-      <origin xyz="0.194763676146297 -0.101665854830299 0.0322193239500774" rpy="0 0 0" />
-      <mass value="2.31657690221752" />
-      <inertia
-        ixx="0.0253400528535679"
-        ixy="0.0764346880668326"
-        ixz="-0.00562954329148165"
-        iyy="0.301489394311443"
-        iyz="0.0021285325929566"
-        izz="0.322973476972127" />
-    </inertial>
-    <visual>
-      <origin xyz="0 0 0" rpy="0 0 0" />
-      <geometry>
-        <mesh filename="package://mars_rover/meshes/RightMainRocker.STL" />
-      </geometry>
-      <material name="">
-        <color rgba="0.792156862745098 0.819607843137255 0.933333333333333 1" />
-      </material>
-    </visual>
-    <collision>
-      <origin xyz="0 0 0" rpy="0 0 0" />
-      <geometry>
-        <mesh filename="package://mars_rover/meshes/RightMainRocker.STL" />
-      </geometry>
-    </collision>
-  </link>
-  <joint name="joint_body_RightMainRocker" type="continuous">
-    <origin xyz="0 -0.155 0.395" rpy="0 0 0" />
-    <parent link="body" />
-    <child link="RightMainRocker" />
-    <axis xyz="0 0 1" />
-  </joint>
-  <link name="RightViceRocker">
-    <inertial>
-      <origin xyz="0 -0.142829300218082 0.00457781208829156" rpy="0 0 0" />
-      <mass value="1.70193743881046" />
-      <inertia
-        ixx="0.0116402353185612"
-        ixy="2.70826203635347E-05"
-        ixz="2.06832199209221E-07"
-        iyy="0.114866898839305"
-        iyz="0.000788350573710642"
-        izz="0.1254823143192" />
-    </inertial>
-    <visual>
-      <origin xyz="0 0 0" rpy="0 0 0" />
-      <geometry>
-        <mesh filename="package://mars_rover/meshes/RightViceRocker.STL" />
-      </geometry>
-      <material name="">
-        <color rgba="0.792156862745098 0.819607843137255 0.933333333333333 1" />
-      </material>
-    </visual>
-    <collision>
-      <origin xyz="0 0 0" rpy="0 0 0" />
-      <geometry>
-        <mesh filename="package://mars_rover/meshes/RightViceRocker.STL" />
-      </geometry>
-    </collision>
-  </link>
-  <joint name="joint_RightMainRocker_RightViceRocker" type="continuous">
-    <origin xyz="-0.40088 -0.023015 0.055" rpy="0 0 0" />
-    <parent link="RightMainRocker" />
-    <child link="RightViceRocker" />
-    <axis xyz="0 0 1" />
-  </joint>
-  <link name="RightMiddleWheel">
-    <inertial>
-      <origin xyz="0 0 0" rpy="0 0 0" />
-      <mass value="2.46800319485063" />
-      <inertia
-        ixx="0.0218761505445029"
-        ixy="-1.9031573010273E-18"
-        ixz="-2.39487588733922E-19"
-        iyy="0.0218761505445029"
-        iyz="-7.04547948608855E-19"
-        izz="0.0405258063947124" />
-    </inertial>
-    <visual>
-      <origin xyz="0 0 0" rpy="0 0 0" />
-      <geometry>
-        <mesh filename="package://mars_rover/meshes/RightMiddleWheel.STL" />
-      </geometry>
-      <material name="">
-        <color rgba="0.792156862745098 0.819607843137255 0.933333333333333 1" />
-      </material>
-    </visual>
-    <collision>
-      <origin xyz="0 0 0" rpy="0 0 0" />
-      <geometry>
-        <mesh filename="package://mars_rover/meshes/RightMiddleWheel.STL" />
-      </geometry>
-    </collision>
-  </link>
-  <joint name="joint_RightViceRocker_RightMiddleWheel" type="continuous">
-    <origin xyz="0.38742 -0.24412 0.09" rpy="${PI} 0 0" />
-    <parent link="RightViceRocker" />
-    <child link="RightMiddleWheel" />
-    <axis xyz="0 0 1" />
-  </joint>
-  <link name="RightRearWheel">
-    <inertial>
-      <origin xyz="0 0 0" rpy="0 0 0" />
-      <mass value="2.46800319485063" />
-      <inertia
-        ixx="0.0218761505445032"
-        ixy="5.55887981239045E-18"
-        ixz="-3.29127182449659E-18"
-        iyy="0.0218761505445032"
-        iyz="1.63702825142094E-18"
-        izz="0.0405258063947131" />
-    </inertial>
-    <visual>
-      <origin xyz="0 0 0" rpy="0 0 0" />
-      <geometry>
-        <mesh filename="package://mars_rover/meshes/RightRearWheel.STL" />
-      </geometry>
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